Commit message: minor

File: robots/panda_arm.xacro (robot description, xacro)
@@ -219,5 +219,5 @@
       <dynamics damping="1.0" friction="0.5"/>
     </joint>
-    <link name="${arm_id}_link8">
+    <!-- <link name="${arm_id}_link8">
       <inertial>
         <origin xyz="0 0 0" rpy="0 0 0"/>
@@ -225,11 +225,39 @@
         <inertia ixx="0.001" ixy="0.0" ixz="0.0" iyy="0.001" iyz="0.0" izz="0.001"/>
       </inertial>
-    </link>
-    <joint name="${arm_id}_joint8" type="fixed">
+    </link> -->
+    <!-- <joint name="${arm_id}_joint8" type="fixed">
     <origin rpy="0 0 0" xyz="0 0 0.107"/>
       <parent link="${arm_id}_link7"/>
       <child link="${arm_id}_link8"/>
       <axis xyz="0 0 0"/>
-    </joint>
+    </joint> -->
+    <link name="${arm_id}_link8">
+      <inertial>
+        <origin xyz="-1.57 0.0 0.0" rpy="0 0 0"/>
+        <mass value="0.0"/>
+        <inertia ixx="0.001" ixy="0.0" ixz="0.0" iyy="0.001" iyz="0.0" izz="0.001"/>
+      </inertial>
+    </link>
+    <joint name="${arm_id}_joint8" type="fixed">
+      <origin rpy="0 0 -0.785398163397" xyz="0 0 0.107"/>
+      <parent link="${arm_id}_link7"/>
+      <child link="${arm_id}_link8"/>
+      <axis xyz="0 0 0"/>
+    </joint>
+  <joint name="ee_fixed_joint" type="fixed">
+    <parent link="panda_link8"/>
+    <child link="ee_link"/>
+    <!--origin rpy="0.0 0.0 1.570796325" xyz="0.0 0.0922 0.0"/-->
+    <!--origin rpy="-1.57 0.0 1.57" xyz="0.0 0. 0.0"/-->
+    <origin rpy="0.0 0.0 -1.57" xyz="0.0 0. 0.1"/>
+  </joint>
+  <link name="ee_link">
+    <collision>
+      <geometry>
+        <box size="0.01 0.01 0.01"/>
+      </geometry>
+      <origin rpy="0 0 0" xyz="0.0 0 0"/>
+    </collision>
+  </link>
   </xacro:macro>
 </robot>

Commit message: initial commit

File: robots/panda_arm.xacro (robot description, xacro)
@@ -219,5 +219,5 @@
       <dynamics damping="1.0" friction="0.5"/>
     </joint>
-    <!-- <link name="${arm_id}_link8">
+    <link name="${arm_id}_link8">
       <inertial>
         <origin xyz="0 0 0" rpy="0 0 0"/>
@@ -225,12 +225,12 @@
         <inertia ixx="0.001" ixy="0.0" ixz="0.0" iyy="0.001" iyz="0.0" izz="0.001"/>
       </inertial>
-    </link> -->
-    <!-- <joint name="${arm_id}_joint8" type="fixed">
+    </link>
+    <joint name="${arm_id}_joint8" type="fixed">
     <origin rpy="0 0 0" xyz="0 0 0.107"/>
       <parent link="${arm_id}_link7"/>
       <child link="${arm_id}_link8"/>
       <axis xyz="0 0 0"/>
-    </joint> -->
-    <link name="${arm_id}_link8">
+    </joint>
+    <!-- <link name="${arm_id}_link8">
       <inertial>
         <origin xyz="-1.57 0.0 0.0" rpy="0 0 0"/>
@@ -238,19 +238,19 @@
         <inertia ixx="0.001" ixy="0.0" ixz="0.0" iyy="0.001" iyz="0.0" izz="0.001"/>
       </inertial>
-    </link>
-    <joint name="${arm_id}_joint8" type="fixed">
+    </link> -->
+    <!-- <joint name="${arm_id}_joint8" type="fixed">
       <origin rpy="0 0 -0.785398163397" xyz="0 0 0.107"/>
       <parent link="${arm_id}_link7"/>
       <child link="${arm_id}_link8"/>
       <axis xyz="0 0 0"/>
-    </joint>
-  <joint name="ee_fixed_joint" type="fixed">
+    </joint> -->
+  <!-- <joint name="ee_fixed_joint" type="fixed">
     <parent link="panda_link8"/>
-    <child link="ee_link"/>
+    <child link="ee_link"/> -->
     <!--origin rpy="0.0 0.0 1.570796325" xyz="0.0 0.0922 0.0"/-->
     <!--origin rpy="-1.57 0.0 1.57" xyz="0.0 0. 0.0"/-->
-    <origin rpy="0.0 0.0 -1.57" xyz="0.0 0. 0.1"/>
-  </joint>
-  <link name="ee_link">
+    <!-- <origin rpy="0.0 0.0 -1.57" xyz="0.0 0. 0.1"/>  -->
+  <!-- </joint> -->
+  <!-- <link name="ee_link">
     <collision>
       <geometry>
@@ -259,5 +259,5 @@
       <origin rpy="0 0 0" xyz="0.0 0 0"/>
     </collision>
-  </link>
+  </link> -->
   </xacro:macro>
 </robot>
