Commit message: tray calibration"

File: robots/franka_panda_no_gripper_tray.urdf (robot description, URDF)
Before this commit: robot panda, 12 links, 11 joints
Joints:
- joint tray_fixed_joint: origin xyz=-0.018 0.023 0.197 rpy=-1.620 -0.003 1.566 -> xyz=0.002 -0.032 0.131 rpy=-1.560 -0.036 1.593

Commit message: tray calibration

File: robots/franka_panda_no_gripper_tray.urdf (robot description, URDF)
Before this commit: robot panda, 12 links, 11 joints
Joints:
- joint tray_fixed_joint: origin xyz=0.002 -0.032 0.131 rpy=-1.560 -0.036 1.593 -> xyz=-0.008 -0.031 0.119 rpy=-1.683 0.039 1.582

Commit message: minor

File: robots/franka_panda_no_gripper_tray.urdf (robot description, URDF)
Before this commit: robot panda, 12 links, 11 joints
Joints:
- joint tray_fixed_joint: origin xyz=-0.008 -0.031 0.119 rpy=-1.683 0.039 1.582 -> xyz=-0.001 -0.018 0.135 rpy=-1.696 -0.062 1.570

Commit message: minor

File: robots/franka_panda_no_gripper_tray.urdf (robot description, URDF)
Before this commit: robot panda, 12 links, 11 joints
Joints:
- joint tray_fixed_joint: origin xyz=-0.001 -0.018 0.135 rpy=-1.696 -0.062 1.570 -> xyz=0.002 -0.039 0.134 rpy=-1.579 -0.035 1.592

Commit message: minor

File: robots/franka_panda_no_gripper_tray.urdf (robot description, URDF)
Before this commit: robot panda, 12 links, 11 joints
Joints:
- joint tray_fixed_joint: origin xyz=0.002 -0.039 0.134 rpy=-1.579 -0.035 1.592 -> xyz=-0.024 0.053 0.205 rpy=-1.627 0.027 1.569

Commit message: new position calibration

File: robots/franka_panda_no_gripper_tray.urdf (robot description, URDF)
Before this commit: robot panda, 12 links, 11 joints
Joints:
- joint tray_fixed_joint: origin xyz=-0.024 0.053 0.205 rpy=-1.627 0.027 1.569 -> xyz=0.003 0.087 0.107 rpy=-1.596 0.004 1.564

Commit message: minor

File: robots/franka_panda_no_gripper_tray.urdf (robot description, URDF)
Before this commit: robot panda, 12 links, 11 joints
Joints:
- joint tray_fixed_joint: origin xyz=0.003 0.087 0.107 rpy=-1.596 0.004 1.564 -> xyz=0.002 0.082 0.106 rpy=-1.593 0.002 1.529

Commit message: minor

File: robots/franka_panda_no_gripper_tray.urdf (robot description, URDF)
Before this commit: robot panda, 12 links, 11 joints
Links:
- link tray_link: geometry collision box size=0.25 0.245 0.04; visual box size=0.25 0.245 0.04
Joints:
- joint tray_fixed_joint: origin xyz=0.002 0.082 0.106 rpy=-1.593 0.002 1.529 -> xyz=0.0 0.125 0.02 rpy=0.0 0.0 0.0
